Commit message: enable odom_tf gazebo only in public sim and laser noise fix

File: omni_base_description/gazebo/gazebo.urdf.xacro (robot description, xacro)
@@ -37,5 +37,10 @@
       <odometryRate>50.0</odometryRate>
       <robotBaseFrame>base_footprint</robotBaseFrame>
-      <publishOdometryTf>true</publishOdometryTf>
+      <xacro:if value="${is_public_sim}">
+        <publishOdometryTf>true</publishOdometryTf>
+      </xacro:if>
+      <xacro:unless value="${is_public_sim}">
+        <publishOdometryTf>false</publishOdometryTf>
+      </xacro:unless>
       <xacro:if value="${is_multiple}">
         <!-- Do something about multirobot -->

File: omni_base_description/robots/omni_base.urdf.xacro (robot description, xacro)
@@ -17,8 +17,10 @@
   <xacro:arg name="rear_laser_model" default="sick-571"/> <!-- false, hokuyo, sick-551, sick-561, sick-571-->
   <xacro:arg name="multiple" default="false"/>
+  <xacro:arg name="public_sim" default="false"/>
   <xacro:arg name="namespace" default=""/>
   <xacro:property name="front_laser_model" value="$(arg front_laser_model)" />
   <xacro:property name="rear_laser_model" value="$(arg rear_laser_model)" />
   <xacro:property name="is_multiple" value="$(arg multiple)" />
+  <xacro:property name="is_public_sim" value="$(arg public_sim)" />
   <xacro:property name="nsp" value="$(arg namespace)" />
   <xacro:if value="${front_laser_model not in ['false', 'sick-551', 'sick-561', 'sick-571', 'hokuyo']}">

File: omni_base_description/urdf/sensors/sick_tim551_laser.gazebo.xacro (robot description, xacro)
@@ -37,5 +37,5 @@
             <type>gaussian</type>
             <mean>0.0</mean>
-            <stddev>0.06</stddev>
+            <stddev>0.008</stddev>
           </noise>
         </ray>

File: omni_base_description/urdf/sensors/sick_tim561_laser.gazebo.xacro (robot description, xacro)
@@ -37,5 +37,5 @@
             <type>gaussian</type>
             <mean>0.0</mean>
-            <stddev>0.06</stddev>
+            <stddev>0.008</stddev>
           </noise>
         </ray>

File: omni_base_description/urdf/sensors/sick_tim571_laser.gazebo.xacro (robot description, xacro)
@@ -37,5 +37,5 @@
             <type>gaussian</type>
             <mean>0.0</mean>
-            <stddev>0.06</stddev>
+            <stddev>0.008</stddev>
           </noise>
         </ray>
