Commit message: swap camera names

File: omni_base_description/urdf/base/base_omni_base_calib.urdf.xacro (robot description, xacro)
@@ -13,9 +13,9 @@
 -->
 <robot xmlns:xacro="http://www.ros.org/wiki/xacro">
-  <xacro:property name="base_rgbd_z" value="0.551436"/>
+  <xacro:property name="roof_rgbd_z" value="0.551436"/>
+  <xacro:property name="roof_rgbd_R" value="0.0"/>
+  <xacro:property name="roof_rgbd_P" value="55.0"/>
+  <xacro:property name="base_rgbd_z" value="0.483197"/>
   <xacro:property name="base_rgbd_R" value="0.0"/>
-  <xacro:property name="base_rgbd_P" value="55.0"/>
-  <xacro:property name="roof_rgbd_z" value="0.483197"/>
-  <xacro:property name="roof_rgbd_R" value="0.0"/>
-  <xacro:property name="roof_rgbd_P" value="12.0"/>
+  <xacro:property name="base_rgbd_P" value="12.0"/>
 </robot>

File: omni_base_description/urdf/sensors/courier.urdf.xacro (robot description, xacro)
@@ -20,12 +20,12 @@
   <!-- spec: rgbd_z, rgbd_R and rgbd_P -->
   <xacro:include filename="${calibration_path}/urdf/base/base_omni_base_calib.urdf.xacro"/>
+  <!-- roof RGBD characteristics -->
+  <xacro:property name="roof_rgbd_x" value="0.327327"/>
+  <xacro:property name="roof_rgbd_y" value="0.0"/>
+  <xacro:property name="roof_rgbd_Y" value="0.0"/>
   <!-- base RGBD characteristics -->
-  <xacro:property name="base_rgbd_x" value="0.327327"/>
+  <xacro:property name="base_rgbd_x" value="0.297329"/>
   <xacro:property name="base_rgbd_y" value="0.0"/>
   <xacro:property name="base_rgbd_Y" value="0.0"/>
-  <!-- roof RGBD characteristics -->
-  <xacro:property name="roof_rgbd_x" value="0.297329"/>
-  <xacro:property name="roof_rgbd_y" value="0.0"/>
-  <xacro:property name="roof_rgbd_Y" value="0.0"/>
   <!-- RGBD base -->
   <xacro:sensor_d435

Commit message: Revert "swap camera names"
This reverts commit 10b11403fde04f52c57782ff8e30f3e92cd042cc.

File: omni_base_description/urdf/base/base_omni_base_calib.urdf.xacro (robot description, xacro)
@@ -13,9 +13,9 @@
 -->
 <robot xmlns:xacro="http://www.ros.org/wiki/xacro">
-  <xacro:property name="roof_rgbd_z" value="0.551436"/>
+  <xacro:property name="base_rgbd_z" value="0.551436"/>
+  <xacro:property name="base_rgbd_R" value="0.0"/>
+  <xacro:property name="base_rgbd_P" value="55.0"/>
+  <xacro:property name="roof_rgbd_z" value="0.483197"/>
   <xacro:property name="roof_rgbd_R" value="0.0"/>
-  <xacro:property name="roof_rgbd_P" value="55.0"/>
-  <xacro:property name="base_rgbd_z" value="0.483197"/>
-  <xacro:property name="base_rgbd_R" value="0.0"/>
-  <xacro:property name="base_rgbd_P" value="12.0"/>
+  <xacro:property name="roof_rgbd_P" value="12.0"/>
 </robot>

File: omni_base_description/urdf/sensors/courier.urdf.xacro (robot description, xacro)
@@ -20,12 +20,12 @@
   <!-- spec: rgbd_z, rgbd_R and rgbd_P -->
   <xacro:include filename="${calibration_path}/urdf/base/base_omni_base_calib.urdf.xacro"/>
+  <!-- base RGBD characteristics -->
+  <xacro:property name="base_rgbd_x" value="0.327327"/>
+  <xacro:property name="base_rgbd_y" value="0.0"/>
+  <xacro:property name="base_rgbd_Y" value="0.0"/>
   <!-- roof RGBD characteristics -->
-  <xacro:property name="roof_rgbd_x" value="0.327327"/>
+  <xacro:property name="roof_rgbd_x" value="0.297329"/>
   <xacro:property name="roof_rgbd_y" value="0.0"/>
   <xacro:property name="roof_rgbd_Y" value="0.0"/>
-  <!-- base RGBD characteristics -->
-  <xacro:property name="base_rgbd_x" value="0.297329"/>
-  <xacro:property name="base_rgbd_y" value="0.0"/>
-  <xacro:property name="base_rgbd_Y" value="0.0"/>
   <!-- RGBD base -->
   <xacro:sensor_d435
