Commit message: Update linters

File: omni_base_description/urdf/base/base.urdf.xacro (robot description, xacro)
@@ -101,8 +101,8 @@
     </joint>
     <!-- Antennas -->
-    <xacro:antenna name="base_antenna_right" parent="base_link" reflect="1">
+    <xacro:antenna name="${name}_antenna_right" parent="${name}_link" reflect="1">
       <origin xyz="-0.2015 -0.13 0.2165" rpy="0 0 0" />
     </xacro:antenna>
-    <xacro:antenna name="base_antenna_left" parent="base_link" reflect="-1">
+    <xacro:antenna name="${name}_antenna_left" parent="${name}_link" reflect="-1">
       <origin xyz="-0.2015 0.13 0.2165" rpy="0 0 0" />
     </xacro:antenna>

File: omni_base_description/urdf/base/base_sensors.urdf.xacro (robot description, xacro)
@@ -52,9 +52,9 @@
   <xacro:macro name="base_sensors" params="name front_laser_model:=sick-561 rear_laser_model:=sick-561 laser_height:=0.13244">
     <!-- Rear Laser Sensor -->
-    <xacro:laser_sensor name="${name}_rear_laser" parent="${name}" model="${rear_laser_model}" ros_topic="scan_rear_raw">
+    <xacro:laser_sensor name="${name}_rear_laser" parent="${name}_link" model="${rear_laser_model}" ros_topic="scan_rear_raw">
       <origin xyz="-0.27512 0.18297 ${laser_height}" rpy="${-180 * deg_to_rad} 0 ${135 * deg_to_rad}" />
     </xacro:laser_sensor>
     <!-- Front Laser Sensor -->
-    <xacro:laser_sensor name="${name}_front_laser" parent="${name}" model="${front_laser_model}" ros_topic="scan_front_raw">
+    <xacro:laser_sensor name="${name}_front_laser" parent="${name}_link" model="${front_laser_model}" ros_topic="scan_front_raw">
       <origin xyz="0.27512 -0.18297 ${laser_height}" rpy="${-180 * deg_to_rad} 0 ${-45 * deg_to_rad}" />
     </xacro:laser_sensor>

File: omni_base_description/urdf/sensors/hokuyo_urg_04lx_ug01_laser.urdf.xacro (robot description, xacro)
@@ -42,5 +42,5 @@
       <axis xyz="0 1 0"/>
       <xacro:insert_block name="origin"/>
-      <parent link="${parent}_link"/>
+      <parent link="${parent}"/>
       <child  link="${name}_link"/>
     </joint>

File: omni_base_description/urdf/sensors/sick_tim551_laser.urdf.xacro (robot description, xacro)
@@ -42,5 +42,5 @@
       <axis xyz="0 1 0"/>
       <xacro:insert_block name="origin"/>
-      <parent link="${parent}_link"/>
+      <parent link="${parent}"/>
       <child  link="${name}_link"/>
     </joint>

File: omni_base_description/urdf/sensors/sick_tim561_laser.urdf.xacro (robot description, xacro)
@@ -42,5 +42,5 @@
       <axis xyz="0 1 0"/>
       <xacro:insert_block name="origin"/>
-      <parent link="${parent}_link"/>
+      <parent link="${parent}"/>
       <child  link="${name}_link"/>
     </joint>

File: omni_base_description/urdf/sensors/sick_tim571_laser.urdf.xacro (robot description, xacro)
@@ -42,5 +42,5 @@
       <axis xyz="0 1 0"/>
       <xacro:insert_block name="origin"/>
-      <parent link="${parent}_link"/>
+      <parent link="${parent}"/>
       <child  link="${name}_link"/>
     </joint>
