Commit message: Fix argument + tests

File: omni_base_description/urdf/sensors/courier.urdf.xacro (robot description, xacro)
@@ -17,5 +17,5 @@
   <xacro:property name="default_calibration_path" value="$(find omni_base_description)"/>
   <xacro:property name="calibration_path" value="$(optenv omni_base_description_calibration_path ${default_calibration_path})"/>
-  <xacro:property name="use_sim" value="$(arg use_sim)" />
+  <xacro:property name="use_sim_time" value="$(arg use_sim_time)" />
   <!-- base RGBD characteristics -->
   <xacro:property name="base_rgbd_x" value="0.327327"/>
@@ -31,4 +31,5 @@
   <!-- spec: rgbd_z, rgbd_R and rgbd_P -->
   <xacro:include filename="${calibration_path}/urdf/base/base_omni_base_calib.urdf.xacro"/>
+  <xacro:include filename="$(find pal_urdf_utils)/urdf/deg_to_rad.urdf.xacro" />
   <!-- RGBD base -->
   <xacro:sensor_d435
@@ -36,5 +37,5 @@
     parent="base_link"
     topics_ns="base_rgbd_camera"
-    use_nominal_extrinsics="${use_sim}">
+    use_nominal_extrinsics="${use_sim_time}">
     <origin
         xyz="${base_rgbd_x}
@@ -50,5 +51,5 @@
     parent="base_link"
     topics_ns="roof_rgbd_camera"
-    use_nominal_extrinsics="${use_sim}">
+    use_nominal_extrinsics="${use_sim_time}">
     <origin
         xyz="${roof_rgbd_x}
