Commit message: added realsense support

File: omni_base_description/robots/omni_base.urdf.xacro (robot description, xacro)
@@ -16,10 +16,13 @@
   <xacro:arg name="front_laser_model" default="sick-571"/> <!-- false, hokuyo, sick-551, sick-561, sick-571-->
   <xacro:arg name="rear_laser_model" default="sick-571"/> <!-- false, hokuyo, sick-551, sick-561, sick-571-->
+  <xacro:arg name="rgbd_sensors" default="false"/> <!-- false, true-->
   <xacro:arg name="multiple" default="false"/>
   <xacro:arg name="public_sim" default="false"/>
+  <xacro:arg name="simulation" default="false"/>
   <xacro:arg name="namespace" default=""/>
   <xacro:arg name="is_public_sim" default="false"/>
   <xacro:property name="front_laser_model" value="$(arg front_laser_model)" />
   <xacro:property name="rear_laser_model" value="$(arg rear_laser_model)" />
+  <xacro:property name="rgbd_sensors" value="$(arg rgbd_sensors)"/>
   <xacro:property name="is_multiple" value="$(arg multiple)" />
   <xacro:property name="is_public_sim" value="$(arg is_public_sim)" />
@@ -43,3 +46,8 @@
   <!-- Now we can start using the macros included above to define the actual robot -->
   <xacro:base_sensors name="base" front_laser_model="$(arg front_laser_model)" rear_laser_model="$(arg rear_laser_model)"/>
+  <!-- RGBD Sensors -->
+  <xacro:if value="${rgbd_sensors}">
+    <xacro:include filename="$(find omni_base_description)/urdf/cameras_add_on/cameras_add_on.urdf.xacro" />
+    <xacro:cameras_add_on name="cameras_add_on" parent="base_link"/>
+  </xacro:if>
 </robot>

Commit message: removed simulation arg and fix use_nominal_extrinsic

File: omni_base_description/robots/omni_base.urdf.xacro (robot description, xacro)
@@ -19,5 +19,4 @@
   <xacro:arg name="multiple" default="false"/>
   <xacro:arg name="public_sim" default="false"/>
-  <xacro:arg name="simulation" default="false"/>
   <xacro:arg name="namespace" default=""/>
   <xacro:arg name="is_public_sim" default="false"/>

File: omni_base_description/urdf/sensors/courier.urdf.xacro (robot description, xacro)
@@ -16,4 +16,5 @@
   <xacro:property name="default_calibration_path" value="$(find omni_base_description)"/>
   <xacro:property name="calibration_path" value="$(optenv omni_base_description_calibration_path ${default_calibration_path})"/>
+  <xacro:property name="use_sim" value="$(arg use_sim)" />
   <!-- base/roof RGBD calibratable characteristics -->
   <!-- spec: rgbd_z, rgbd_R and rgbd_P -->
@@ -32,5 +33,5 @@
     parent="base_link"
     topics_ns="base_rgbd_camera"
-    use_nominal_extrinsics="${simulation}">
+    use_nominal_extrinsics="${use_sim}">
     <origin
         xyz="${base_rgbd_x}
@@ -46,5 +47,5 @@
     parent="base_link"
     topics_ns="roof_rgbd_camera"
-    use_nominal_extrinsics="${simulation}">
+    use_nominal_extrinsics="${use_sim}">
     <origin
         xyz="${roof_rgbd_x}

Commit message: add missing argument is_public_sim

File: omni_base_description/robots/omni_base.urdf.xacro (robot description, xacro)
@@ -19,8 +19,9 @@
   <xacro:arg name="public_sim" default="false"/>
   <xacro:arg name="namespace" default=""/>
+  <xacro:arg name="is_public_sim" default="false"/>
   <xacro:property name="front_laser_model" value="$(arg front_laser_model)" />
   <xacro:property name="rear_laser_model" value="$(arg rear_laser_model)" />
   <xacro:property name="is_multiple" value="$(arg multiple)" />
-  <xacro:property name="is_public_sim" value="$(arg public_sim)" />
+  <xacro:property name="is_public_sim" value="$(arg is_public_sim)" />
   <xacro:property name="nsp" value="$(arg namespace)" />
   <xacro:if value="${front_laser_model not in ['false', 'sick-551', 'sick-561', 'sick-571', 'hokuyo']}">
