Commit message: Standardize urdf + update lauch args

File: omni_base_description/robots/omni_base.urdf.xacro (robot description, xacro)
@@ -1,5 +1,5 @@
 <?xml version="1.0"?>
 <!--
-  Copyright (c) 2023 PAL Robotics S.L. All rights reserved.
+  Copyright (c) 2024 PAL Robotics S.L. All rights reserved.
   Licensed under the Apache License, Version 2.0 (the "License");
   you may not use this file except in compliance with the License.
@@ -11,20 +11,24 @@
   See the License for the specific language governing permissions and
   limitations under the License.
- -->
+-->
 <robot  xmlns:xacro="http://ros.org/wiki/xacro" name="omni_base" >
-  <xacro:arg name="use_sim" default="false"/>
-  <xacro:arg name="front_laser_model" default="sick-571"/> <!-- false, hokuyo, sick-551, sick-561, sick-571-->
-  <xacro:arg name="rear_laser_model" default="sick-571"/> <!-- false, hokuyo, sick-551, sick-561, sick-571-->
-  <xacro:arg name="rgbd_sensors" default="false"/> <!-- false, true-->
-  <xacro:arg name="multiple" default="false"/>
-  <xacro:arg name="public_sim" default="false"/>
+  <!-- ARGUMENTS -->
+  <!-- false, hokuyo, sick-551, sick-561, sick-571-->
+  <xacro:arg name="front_laser_model" default="sick-571"/>
+  <!-- false, hokuyo, sick-551, sick-561, sick-571-->
+  <xacro:arg name="rear_laser_model" default="sick-571"/>
+  <!-- false, true-->
+  <xacro:arg name="rgbd_sensors" default="false"/>
+  <!-- Execution env config -->
+  <xacro:arg name="use_sim_time" default="false"/>
+  <xacro:arg name="is_multiple" default="false"/>
   <xacro:arg name="namespace" default=""/>
   <xacro:arg name="is_public_sim" default="false"/>
+  <!-- PROPERTIES -->
+  <!-- HW configuration -->
   <xacro:property name="front_laser_model" value="$(arg front_laser_model)" />
   <xacro:property name="rear_laser_model" value="$(arg rear_laser_model)" />
   <xacro:property name="rgbd_sensors" value="$(arg rgbd_sensors)"/>
-  <xacro:property name="is_multiple" value="$(arg multiple)" />
-  <xacro:property name="is_public_sim" value="$(arg is_public_sim)" />
-  <xacro:property name="nsp" value="$(arg namespace)" />
+  <!-- HW configuration check -->
   <xacro:if value="${front_laser_model not in ['false', 'sick-551', 'sick-561', 'sick-571', 'hokuyo']}">
     <xacro:wrong_laser_model/>
@@ -33,19 +37,28 @@
     <xacro:wrong_laser_model/>
   </xacro:if>
-  <!-- The following included files set up definitions of parts of the robot body -->
+  <!-- Execution env configuration -->
+  <xacro:property name="use_sim_time" default="$(arg use_sim_time)"/>
+  <xacro:property name="is_multiple" value="$(arg is_multiple)" />
+  <xacro:property name="namespace" value="$(arg namespace)" />
+  <xacro:property name="is_public_sim" value="$(arg is_public_sim)" />
+  <!-- INCLUDES -->
   <!-- Base -->
   <xacro:include filename="$(find omni_base_description)/urdf/base/base_sensors.urdf.xacro" />
-  <!-- Generic simulator_gazebo plugins -->
-  <xacro:include filename="$(find omni_base_description)/gazebo/gazebo.urdf.xacro" />
-  <!-- ros2_control -->
+  <!-- RGBD Sensors -->
+  <xacro:if value="${rgbd_sensors}">
+    <xacro:include filename="$(find omni_base_description)/urdf/cameras_add_on/cameras_add_on.urdf.xacro" />
+  </xacro:if>
+  <!-- Materials for visualization -->
+  <xacro:include filename="$(find pal_urdf_utils)/urdf/materials.urdf.xacro" />
+  <!-- Utils for degree to radian conversion -->
+  <xacro:include filename="$(find pal_urdf_utils)/urdf/deg_to_rad.urdf.xacro" />
+  <!-- ROS 2 Control -->
   <xacro:include filename="$(find omni_base_description)/ros2_control/ros2_control.urdf.xacro" />
-  <xacro:omni_base_ros2_control use_sim="$(arg use_sim)" />
-  <!-- Materials for visualization -->
-  <xacro:include filename="$(find omni_base_description)/urdf/materials.urdf.xacro" />
+  <xacro:omni_base_ros2_control />
+  <!-- ROBOT DEFINITION -->
   <!-- Now we can start using the macros included above to define the actual robot -->
   <xacro:base_sensors name="base" front_laser_model="$(arg front_laser_model)" rear_laser_model="$(arg rear_laser_model)"/>
   <!-- RGBD Sensors -->
   <xacro:if value="${rgbd_sensors}">
-    <xacro:include filename="$(find omni_base_description)/urdf/cameras_add_on/cameras_add_on.urdf.xacro" />
     <xacro:cameras_add_on name="cameras_add_on" parent="base_link"/>
   </xacro:if>

File: omni_base_description/ros2_control/ros2_control.urdf.xacro (robot description, xacro)
@@ -1,5 +1,5 @@
 <?xml version="1.0"?>
 <!--
-Copyright (c) 2023 PAL Robotics S.L. All rights reserved.
+Copyright (c) 2024 PAL Robotics S.L. All rights reserved.
 Licensed under the Apache License, Version 2.0 (the "License");
 you may not use this file except in compliance with the License.
@@ -12,17 +12,33 @@
 limitations under the License.
  -->
-<robot xmlns:xacro="http://ros.org/wiki/xacro"
-       name="omni_base" >
-<xacro:macro name="omni_base_ros2_control" params="use_sim:=^|false">
-    <xacro:include filename="$(find omni_base_description)/urdf/wheels/wheel.ros2_control.xacro"/>
-    <xacro:include filename="$(find omni_base_description)/urdf/sensors/sensors.ros2_control.xacro"/>
+<robot xmlns:xacro="http://ros.org/wiki/xacro" name="omni_base" >
+  <!-- INCLUDES -->
+  <xacro:include filename="$(find omni_base_description)/urdf/wheels/wheel.ros2_control.xacro"/>
+  <xacro:include filename="$(find omni_base_description)/urdf/sensors/sensors.ros2_control.xacro"/>
+  <!-- MACRO DEFINITION-->
+  <xacro:macro name="omni_base_ros2_control">
+    <!-- Init the ROS 2 control gazebo interface -->
+    <xacro:if value="${use_sim_time}">
+      <gazebo>
+        <plugin filename="libgazebo_ros2_control.so" name="gazebo_ros2_control">
+          <parameters>$(find omni_base_description)/ros2_control/gazebo_controller_manager_cfg.yaml</parameters>
+          <robot_sim_type>gazebo_ros2_control/GazeboSystem</robot_sim_type>
+          <control_period>0.001</control_period>
+        </plugin>
+      </gazebo>
+    </xacro:if>
+    <!-- ROS 2 control config-->
     <ros2_control name="ros2_control_omni_base_system" type="system">
-      <xacro:if value="$(arg use_sim)">
-        <xacro:ros2_control_imu name="base_imu_sensor"/>
+      <!-- Execution env config -->
+      <xacro:if value="${use_sim_time}">
+        <!-- HW interface: gazebo-->
         <hardware>
           <plugin>gazebo_ros2_control/GazeboSystem</plugin>
         </hardware>
+        <!-- IMU sensor (only in simulation)-->
+        <xacro:ros2_control_imu name="base_imu_sensor"/>
       </xacro:if>
-      <xacro:unless value="$(arg use_sim)">
+      <xacro:unless value="${use_sim_time}">
+        <!-- HW interface: robot control-->
         <hardware>
           <plugin>robot_control/RobotControl</plugin>

File: omni_base_description/urdf/base/antenna.urdf.xacro (robot description, xacro)
@@ -13,4 +13,5 @@
 -->
 <robot xmlns:xacro="http://ros.org/wiki/xacro">
+  <!-- MACRO DEFINITION -->
   <xacro:macro name="antenna" params="name parent *origin reflect:=1">
     <link name="${name}_link">

File: omni_base_description/urdf/base/base.urdf.xacro (robot description, xacro)
@@ -1,5 +1,5 @@
 <?xml version="1.0"?>
 <!--
-  Copyright (c) 2023 PAL Robotics S.L. All rights reserved.
+  Copyright (c) 2024 PAL Robotics S.L. All rights reserved.
   Licensed under the Apache License, Version 2.0 (the "License");
   you may not use this file except in compliance with the License.
@@ -11,10 +11,7 @@
   See the License for the specific language governing permissions and
   limitations under the License.
- -->
+-->
 <robot xmlns:xacro="http://ros.org/wiki/xacro">
-  <xacro:include filename="$(find omni_base_description)/urdf/deg_to_rad.xacro"/>
-  <xacro:include filename="$(find omni_base_description)/urdf/wheels/wheel.urdf.xacro"/>
-  <xacro:include filename="$(find omni_base_description)/urdf/base/antenna.urdf.xacro"/>
-  <xacro:include filename="$(find omni_base_description)/urdf/sensors/imu.urdf.xacro"/>
+  <!-- PROPERTIES -->
   <!-- Wheel characteristics -->
   <xacro:property name="wheel_radius"     value="0.0762"/>
@@ -25,6 +22,10 @@
   <xacro:property name="wheel_velocity"   value="1.0"/>
   <xacro:property name="suspension_sagital_separation" value="0.345"/>
+  <!-- INCLUDES -->
+  <xacro:include filename="$(find omni_base_description)/urdf/wheels/wheel.urdf.xacro"/>
+  <xacro:include filename="$(find omni_base_description)/urdf/base/antenna.urdf.xacro"/>
+  <!-- MACRO DEFINITION-->
   <xacro:macro name="base" params="name">
-    <!-- Base footprint -->
+    <!-- Base -->
     <link name="${name}_link">
       <inertial>
@@ -62,4 +63,5 @@
       </collision>
     </link>
+    <!-- Base footprint -->
     <link name="${name}_footprint"/>
     <joint name="${name}_footprint_joint" type="fixed">
@@ -68,19 +70,4 @@
       <parent link="${name}_footprint"/>
     </joint>
-  <!-- gazebo parameters are given here for base_link through base_footprint -->
-    <gazebo reference="${name}_footprint">
-      <kp>100000000.0</kp>
-      <kd>10.0</kd>
-      <mu1>0.1</mu1>
-      <mu2>0.1</mu2>
-      <fdir1>1 0 0</fdir1>
-      <maxVel>10.0</maxVel>
-      <minDepth>0.0005</minDepth>
-      <laserRetro>0</laserRetro>
-    </gazebo>
-    <!-- IMU -->
-    <xacro:imu_sensor name="${name}_imu" parent="${name}_link" update_rate="100.0">
-      <origin xyz="-0.287 0 0.092163" rpy="0 0 ${90.0 * deg_to_rad}" />
-    </xacro:imu_sensor>
     <!-- Docking link -->
     <link name="${name}_dock_link">

File: omni_base_description/urdf/base/base_omni_base_calib.urdf.xacro (robot description, xacro)
@@ -13,7 +13,10 @@
 -->
 <robot xmlns:xacro="http://www.ros.org/wiki/xacro">
+  <!-- PROPERTIES -->
+  <!-- RGBD base -->
   <xacro:property name="base_rgbd_z" value="0.551436"/>
   <xacro:property name="base_rgbd_R" value="0.0"/>
   <xacro:property name="base_rgbd_P" value="55.0"/>
+  <!-- RGBD roof -->
   <xacro:property name="roof_rgbd_z" value="0.483197"/>
   <xacro:property name="roof_rgbd_R" value="0.0"/>

File: omni_base_description/urdf/base/base_sensors.urdf.xacro (robot description, xacro)
@@ -13,14 +13,15 @@
  -->
 <robot xmlns:xacro="http://ros.org/wiki/xacro">
+  <!-- INCLUDES -->
   <xacro:include filename="$(find omni_base_description)/urdf/base/base.urdf.xacro"/>
+  <xacro:include filename="$(find omni_base_description)/urdf/sensors/imu.urdf.xacro"/>
   <xacro:include filename="$(find omni_base_description)/urdf/sensors/hokuyo_urg_04lx_ug01_laser.urdf.xacro"/>
   <xacro:include filename="$(find omni_base_description)/urdf/sensors/sick_tim551_laser.urdf.xacro"/>
   <xacro:include filename="$(find omni_base_description)/urdf/sensors/sick_tim561_laser.urdf.xacro"/>
   <xacro:include filename="$(find omni_base_description)/urdf/sensors/sick_tim571_laser.urdf.xacro"/>
-  <xacro:include filename="$(find omni_base_description)/urdf/deg_to_rad.xacro"/>
-  <!-- Laser model can be; false, hokuyo, sick-551, sick-561, sick-571-->
+  <!-- LASER MACRO DEFINITION -->
   <xacro:macro name="laser_sensor" params="name parent model ros_topic *origin update_rate:=10">
     <xacro:if value="${model == 'sick-551'}">
-      <!-- Rear Laser;  Theoretic FOV = 270 -->
+      <!-- Rear Laser:  Theoretic FOV = 270 -->
       <xacro:sick_tim551_laser name="${name}" parent="${parent}" ros_topic="${ros_topic}" update_rate="${update_rate}" min_angle="${-135 * deg_to_rad}" max_angle="${135 * deg_to_rad}" >
         <xacro:insert_block name="origin" />
@@ -28,5 +29,5 @@
     </xacro:if>
     <xacro:if value="${model == 'sick-561'}">
-      <!-- Rear Laser;  Theoretic FOV = 270 -->
+      <!-- Rear Laser:  Theoretic FOV = 270 -->
       <xacro:sick_tim561_laser name="${name}" parent="${parent}" ros_topic="${ros_topic}" update_rate="${update_rate}" min_angle="${-135 * deg_to_rad}" max_angle="${135 * deg_to_rad}" >
         <xacro:insert_block name="origin" />
@@ -34,5 +35,5 @@
     </xacro:if>
     <xacro:if value="${model == 'sick-571'}">
-      <!-- Rear Laser;  Theoretic FOV = 270 -->
+      <!-- Rear Laser:  Theoretic FOV = 270 -->
       <xacro:sick_tim571_laser name="${name}" parent="${parent}" ros_topic="${ros_topic}" update_rate="${update_rate}" min_angle="${-135 * deg_to_rad}" max_angle="${135 * deg_to_rad}" >
         <xacro:insert_block name="origin" />
@@ -40,5 +41,5 @@
     </xacro:if>
     <xacro:if value="${model == 'hokuyo'}">
-      <!-- Rear Laser;  Theoretic FOV = 240 -->
+      <!-- Rear Laser:  Theoretic FOV = 240 -->
       <xacro:hokuyo_urg_04lx_ug01_laser name="${name}" parent="${parent}" ros_topic="${ros_topic}" update_rate="${update_rate}" min_angle="${-120 * deg_to_rad}" max_angle="${120 * deg_to_rad}" >
         <xacro:insert_block name="origin" />
@@ -46,7 +47,8 @@
     </xacro:if>
   </xacro:macro>
-  <!-- front_laser_model can be; false, hokuyo, sick-551, sick-561, sick-571-->
-  <!-- rear_laser_model can be; false, hokuyo, sick-551, sick-561, sick-571-->
-  <xacro:macro name="base_sensors" params=" name front_laser_model:=sick-561 rear_laser_model:=sick-561 laser_height:=0.13244">
+  <!-- MACRO DEFINITION -->
+  <!-- front_laser_model can be: false, hokuyo, sick-551, sick-561, sick-571-->
+  <!-- rear_laser_model can be: false, hokuyo, sick-551, sick-561, sick-571-->
+  <xacro:macro name="base_sensors" params="name front_laser_model:=sick-561 rear_laser_model:=sick-561 laser_height:=0.13244">
     <!-- Rear Laser Sensor -->
     <xacro:laser_sensor name="${name}_rear_laser" parent="${name}" model="${rear_laser_model}" ros_topic="scan_rear_raw">
@@ -70,4 +72,8 @@
         </inertial>
     </link>
+    <!-- IMU -->
+    <xacro:imu_sensor name="${name}_imu" parent="${name}_link" update_rate="100.0">
+      <origin xyz="-0.287 0 0.092163" rpy="0 0 ${90.0 * deg_to_rad}" />
+    </xacro:imu_sensor>
     <xacro:base name="${name}"/>
   </xacro:macro>

File: omni_base_description/urdf/cameras_add_on/cameras_add_on.urdf.xacro (robot description, xacro)
@@ -13,6 +13,5 @@
 -->
 <robot xmlns:xacro="http://ros.org/wiki/xacro">
-  <!--File includes-->
-  <xacro:include filename="$(find omni_base_description)/urdf/deg_to_rad.xacro" />
+  <!-- MACRO DEFINITION -->
   <xacro:macro name="cameras_add_on" params="name parent">
     <link name="${name}_link">

File: omni_base_description/urdf/sensors/courier.urdf.xacro (robot description, xacro)
@@ -13,11 +13,9 @@
 -->
 <robot xmlns:xacro="http://ros.org/wiki/xacro">
-  <xacro:include filename="$(find realsense2_description)/urdf/_d435.urdf.xacro" />
+  <!-- PROPERTIES -->
+  <!-- Execution env config -->
   <xacro:property name="default_calibration_path" value="$(find omni_base_description)"/>
   <xacro:property name="calibration_path" value="$(optenv omni_base_description_calibration_path ${default_calibration_path})"/>
   <xacro:property name="use_sim" value="$(arg use_sim)" />
-  <!-- base/roof RGBD calibratable characteristics -->
-  <!-- spec; rgbd_z, rgbd_R and rgbd_P -->
-  <xacro:include filename="${calibration_path}/urdf/base/base_omni_base_calib.urdf.xacro"/>
   <!-- base RGBD characteristics -->
   <xacro:property name="base_rgbd_x" value="0.327327"/>
@@ -28,4 +26,9 @@
   <xacro:property name="roof_rgbd_y" value="0.0"/>
   <xacro:property name="roof_rgbd_Y" value="0.0"/>
+  <!-- INCLUDES -->
+  <xacro:include filename="$(find realsense2_description)/urdf/_d435.urdf.xacro" />
+  <!-- base/roof RGBD calibratable characteristics -->
+  <!-- spec: rgbd_z, rgbd_R and rgbd_P -->
+  <xacro:include filename="${calibration_path}/urdf/base/base_omni_base_calib.urdf.xacro"/>
   <!-- RGBD base -->
   <xacro:sensor_d435

File: omni_base_description/urdf/sensors/hokuyo_urg_04lx_ug01_laser.urdf.xacro (robot description, xacro)
@@ -13,5 +13,7 @@
  -->
 <robot xmlns:xacro="http://ros.org/wiki/xacro">
+  <!-- INCLUDES -->
   <xacro:include filename="$(find omni_base_description)/urdf/sensors/hokuyo_urg_04lx_ug01_laser.gazebo.xacro" />
+  <!-- MACRO DEFINITION -->
   <xacro:macro name="hokuyo_urg_04lx_ug01_laser" params="name parent *origin ros_topic update_rate min_angle max_angle">
     <link name="${name}_link" type="laser">
@@ -43,5 +45,5 @@
       <child  link="${name}_link"/>
     </joint>
-    <!-- gazebo extensions -->
+    <!-- Gazebo config -->
     <xacro:hokuyo_urg_04lx_ug01_laser_gazebo name="${name}" ros_topic="${ros_topic}" update_rate="${update_rate}" min_angle="${min_angle}" max_angle="${max_angle}" />
   </xacro:macro>

File: omni_base_description/urdf/sensors/sick_tim551_laser.gazebo.xacro (robot description, xacro)
@@ -13,4 +13,5 @@
  -->
 <robot xmlns:xacro="http://ros.org/wiki/xacro">
+  <!-- MACRO DEFINITION -->
   <xacro:macro name="sick_tim551_laser_gazebo" params="name ros_topic update_rate min_angle max_angle">
     <gazebo reference="${name}_link">

File: omni_base_description/urdf/sensors/sick_tim551_laser.urdf.xacro (robot description, xacro)
@@ -13,5 +13,7 @@
  -->
 <robot xmlns:xacro="http://ros.org/wiki/xacro">
+  <!-- INCLUDES -->
   <xacro:include filename="$(find omni_base_description)/urdf/sensors/sick_tim551_laser.gazebo.xacro" />
+  <!-- MACRO DEFINITION -->
   <xacro:macro name="sick_tim551_laser" params="name parent *origin ros_topic update_rate min_angle max_angle">
      <link name="${name}_link" type="laser">

File: omni_base_description/urdf/sensors/sick_tim561_laser.gazebo.xacro (robot description, xacro)
@@ -13,4 +13,5 @@
  -->
 <robot xmlns:xacro="http://ros.org/wiki/xacro">
+  <!-- MACRO DEFINITION -->
   <xacro:macro name="sick_tim561_laser_gazebo" params="name ros_topic update_rate min_angle max_angle">
     <gazebo reference="${name}_link">

File: omni_base_description/urdf/sensors/sick_tim561_laser.urdf.xacro (robot description, xacro)
@@ -13,5 +13,7 @@
  -->
 <robot xmlns:xacro="http://ros.org/wiki/xacro">
+  <!-- INCLUDES -->
   <xacro:include filename="$(find omni_base_description)/urdf/sensors/sick_tim561_laser.gazebo.xacro" />
+  <!-- MACRO DEFINITION -->
   <xacro:macro name="sick_tim561_laser" params="name parent *origin ros_topic update_rate min_angle max_angle">
      <link name="${name}_link" type="laser">

File: omni_base_description/urdf/sensors/sick_tim571_laser.gazebo.xacro (robot description, xacro)
@@ -13,4 +13,5 @@
  -->
 <robot xmlns:xacro="http://ros.org/wiki/xacro">
+  <!-- MACRO DEFINITION -->
   <xacro:macro name="sick_tim571_laser_gazebo" params="name ros_topic update_rate min_angle max_angle">
     <gazebo reference="${name}_link">

File: omni_base_description/urdf/sensors/sick_tim571_laser.urdf.xacro (robot description, xacro)
@@ -13,5 +13,7 @@
  -->
 <robot xmlns:xacro="http://ros.org/wiki/xacro">
+  <!-- INCLUDES -->
   <xacro:include filename="$(find omni_base_description)/urdf/sensors/sick_tim571_laser.gazebo.xacro" />
+  <!-- MACRO DEFINITION -->
   <xacro:macro name="sick_tim571_laser" params="name parent *origin ros_topic update_rate min_angle max_angle">
      <link name="${name}_link" type="laser">

File: omni_base_description/urdf/wheels/wheel.urdf.xacro (robot description, xacro)
@@ -13,8 +13,9 @@
  -->
 <robot xmlns:xacro="http://ros.org/wiki/xacro">
-  <xacro:property name="PI" value="3.1415926535897931" />
+  <!-- INCLUDES -->
   <xacro:include filename="$(find omni_base_description)/urdf/wheels/wheel.gazebo.xacro"/>
-  <!-- frontal_reflect; front; +1 and rear; -1 -->
-  <!-- sagital_reflect; right; +1 and left; -1 -->
+  <!-- MACRO DEFINITION -->
+  <!-- frontal_reflect: front: +1 and rear: -1 -->
+  <!-- sagital_reflect: right: +1 and left: -1 -->
   <xacro:macro name="wheel" params="side parent sagital_reflect frontal_reflect radius width torque velocity sagital_separation frontal_separation">
     <link name="suspension_${side}_link">

Commit message: Change rgbd sensors to add-on-module

File: omni_base_description/robots/omni_base.urdf.xacro (robot description, xacro)
@@ -19,5 +19,5 @@
   <xacro:arg name="rear_laser_model" default="sick-571"/>
   <!-- false, true-->
-  <xacro:arg name="rgbd_sensors" default="false"/>
+  <xacro:arg name="add_on_module" default="no-add-on"/>
   <!-- Execution env config -->
   <xacro:arg name="use_sim_time" default="false"/>
@@ -29,5 +29,5 @@
   <xacro:property name="front_laser_model" value="$(arg front_laser_model)" />
   <xacro:property name="rear_laser_model" value="$(arg rear_laser_model)" />
-  <xacro:property name="rgbd_sensors" value="$(arg rgbd_sensors)"/>
+  <xacro:property name="add_on_module" value="$(arg add_on_module)"/>
   <!-- HW configuration check -->
   <xacro:if value="${front_laser_model not in ['no-laser', 'sick-551', 'sick-561', 'sick-571', 'hokuyo']}">
@@ -36,4 +36,7 @@
   <xacro:if value="${rear_laser_model not in ['no-laser', 'sick-551', 'sick-561', 'sick-571', 'hokuyo']}">
     <xacro:wrong_laser_model/>
+  </xacro:if>
+  <xacro:if value="${add_on_module not in ['no-add-on', 'rgbd-sensors']}">
+    <xacro:wrong_add_on_module/>
   </xacro:if>
   <!-- Execution env configuration -->
@@ -46,5 +49,5 @@
   <xacro:include filename="$(find omni_base_description)/urdf/base/base_sensors.urdf.xacro" />
   <!-- RGBD Sensors -->
-  <xacro:if value="${rgbd_sensors}">
+  <xacro:if value="${add_on_module == 'rgbd-sensors'}">
     <xacro:include filename="$(find omni_base_description)/urdf/cameras_add_on/cameras_add_on.urdf.xacro" />
   </xacro:if>
@@ -60,5 +63,5 @@
   <xacro:base_sensors name="base" front_laser_model="$(arg front_laser_model)" rear_laser_model="$(arg rear_laser_model)"/>
   <!-- RGBD Sensors -->
-  <xacro:if value="${rgbd_sensors}">
+  <xacro:if value="${add_on_module == 'rgbd-sensors'}">
     <xacro:cameras_add_on name="cameras_add_on" parent="base_link"/>
   </xacro:if>
