Commit message: Harmonic
Signed-off-by: Juancams <jc.manzanares.serrano@gmail.com>

File: omni_base_description/ros2_control/ros2_control.urdf.xacro (robot description, xacro)
@@ -21,5 +21,5 @@
     <xacro:if value="${use_sim_time}">
       <gazebo>
-        <plugin filename="libgazebo_ros2_control.so" name="gazebo_ros2_control">
+        <plugin filename="libgz_ros2_control-system.so" name="gz_ros2_control::GazeboSimROS2ControlPlugin">
           <parameters>$(find omni_base_description)/ros2_control/gazebo_controller_manager_cfg.yaml</parameters>
           <!-- <robot_sim_type>gazebo_ros2_control/GazeboSystem</robot_sim_type>
@@ -34,5 +34,5 @@
         <!-- HW interface; gazebo-->
         <hardware>
-          <plugin>gazebo_ros2_control/GazeboSystem</plugin>
+          <plugin>gz_ros2_control/GazeboSimSystem</plugin>
         </hardware>
         <!-- IMU sensor (only in simulation)-->

File: omni_base_description/urdf/base/base.urdf.xacro (robot description, xacro)
@@ -40,5 +40,5 @@
         <origin xyz="0 0 0" rpy="0 0 0" />
         <geometry>
-          <mesh filename="package://omni_base_description/meshes/base/base_link.stl" />
+          <mesh filename="file://$(find omni_base_description)/meshes/base/base_link.stl" />
         </geometry>
         <material name="">
@@ -83,5 +83,5 @@
         <origin xyz="0 0 0" rpy="0 0 0" />
         <geometry>
-          <mesh filename="package://omni_base_description/meshes/base/base_dock_link.stl" />
+          <mesh filename="file://$(find omni_base_description)/meshes/base/base_dock_link.stl" />
         </geometry>
         <material name="">
@@ -92,5 +92,5 @@
         <origin xyz="0 0 0" rpy="0 0 0" />
         <geometry>
-          <mesh filename="package://omni_base_description/meshes/base/base_dock_link.stl" />
+          <mesh filename="file://$(find omni_base_description)/meshes/base/base_dock_link.stl" />
         </geometry>
       </collision>

File: omni_base_description/urdf/cameras_add_on/cameras_add_on.urdf.xacro (robot description, xacro)
@@ -26,5 +26,5 @@
           <origin xyz="0 0 -0.04" rpy="1.57 0 1.57"/>
           <geometry>
-            <mesh filename="package://omni_base_description/meshes/cameras_add_on/cameras_add_on.stl" scale="1 1 1"/>
+            <mesh filename="file://$(find omni_base_description)/meshes/cameras_add_on/cameras_add_on.stl" scale="1 1 1"/>
           </geometry>
           <material name="White" />
@@ -33,5 +33,5 @@
           <origin xyz="0 0 -0.04" rpy="1.57 0 1.57"/>
           <geometry>
-            <mesh filename="package://omni_base_description/meshes/cameras_add_on/cameras_add_on.stl" scale="1 1 1"/>
+            <mesh filename="file://$(find omni_base_description)/meshes/cameras_add_on/cameras_add_on.stl" scale="1 1 1"/>
           </geometry>
           <material name="White" />

File: omni_base_description/urdf/objects/antenna.urdf.xacro (robot description, xacro)
@@ -25,5 +25,5 @@
         <origin xyz="0 0 0" rpy="0 0 0" />
         <geometry>
-          <mesh filename="package://omni_base_description/meshes/base/base_antena_link.stl" scale="1 ${reflect} 1" />
+          <mesh filename="file://$(find omni_base_description)/meshes/base/base_antena_link.stl" scale="1 ${reflect} 1" />
         </geometry>
         <material name="">
@@ -34,5 +34,5 @@
         <origin xyz="0 0 0" rpy="0 0 0" />
         <geometry>
-          <mesh filename="package://omni_base_description/meshes/base/base_antena_link.stl" scale="1 ${reflect} 1"/>
+          <mesh filename="file://$(find omni_base_description)/meshes/base/base_antena_link.stl" scale="1 ${reflect} 1"/>
         </geometry>
       </collision>

File: omni_base_description/urdf/sensors/hokuyo_urg_04lx_ug01_laser.gazebo.xacro (robot description, xacro)
@@ -16,9 +16,11 @@
   <xacro:macro name="hokuyo_urg_04lx_ug01_laser_gazebo" params="name ros_topic update_rate min_angle max_angle">
     <gazebo reference="${name}_link">
-      <sensor type="gpu_ray" name="${name}">
+      <sensor type="gpu_lidar" name="${name}">
         <pose>0 0 0 0 0 0</pose>
         <update_rate>${update_rate}</update_rate>
         <visualize>true</visualize>
-        <ray>
+        <topic>${ros_topic}</topic>
+        <gz_frame_id>${name}_link</gz_frame_id>
+        <lidar>
           <scan>
             <horizontal>
@@ -40,12 +42,5 @@
             <stddev>0.03</stddev>
           </noise>
-        </ray>
-      	<plugin name="${name}" filename="libgazebo_ros_ray_sensor.so">
-          <ros>
-      	    <remapping>~/out:=${ros_topic}</remapping>
-          </ros>
-          <output_type>sensor_msgs/LaserScan</output_type>
-      	  <frame_name>${name}_link</frame_name>
-        </plugin>
+        </lidar>
       </sensor>
       <material>Gazebo/DarkGrey</material>

File: omni_base_description/urdf/sensors/hokuyo_urg_04lx_ug01_laser.urdf.xacro (robot description, xacro)
@@ -28,5 +28,5 @@
         <origin xyz="0 0 0" rpy="0 0 0" />
         <geometry>
-          <mesh filename="package://omni_base_description/meshes/sensors/hokuyo_urg_04lx_ug01.stl"/>
+          <mesh filename="file://$(find omni_base_description)/meshes/sensors/hokuyo_urg_04lx_ug01.stl"/>
         </geometry>
         <material name="DarkGrey"/>

File: omni_base_description/urdf/sensors/imu.gazebo.xacro (robot description, xacro)
@@ -19,4 +19,5 @@
         <always_on>1</always_on>
         <update_rate>${update_rate}</update_rate>
+        <topic>base_imu</topic>
         <imu>
           <noise>
@@ -36,10 +37,4 @@
           </noise>
         </imu>
-        <plugin name="base_imu" filename="libgazebo_ros_imu_sensor.so">
-          <ros>
-            <!-- publish to /imu/data -->
-            <remapping>~/out:=base_imu</remapping>
-          </ros>
-        </plugin>
       </sensor>
     </gazebo>

File: omni_base_description/urdf/sensors/sick_tim551_laser.gazebo.xacro (robot description, xacro)
@@ -16,9 +16,11 @@
   <xacro:macro name="sick_tim551_laser_gazebo" params="name ros_topic update_rate min_angle max_angle">
     <gazebo reference="${name}_link">
-      <sensor type="gpu_ray" name="${name}">
+      <sensor type="gpu_lidar" name="${name}">
         <pose>0 0 0 0 0 0</pose>
         <update_rate>${update_rate}</update_rate>
         <visualize>true</visualize>
-        <ray>
+        <topic>${ros_topic}</topic>
+        <gz_frame_id>${name}_link</gz_frame_id>
+        <lidar>
           <scan>
             <horizontal>
@@ -40,12 +42,5 @@
             <stddev>0.01</stddev>
           </noise>
-        </ray>
-      	<plugin name="${name}" filename="libgazebo_ros_ray_sensor.so">
-          <ros>
-      	    <remapping>~/out:=${ros_topic}</remapping>
-          </ros>
-          <output_type>sensor_msgs/LaserScan</output_type>
-      	  <frame_name>${name}_link</frame_name>
-        </plugin>
+        </lidar>
       </sensor>
       <material>Gazebo/DarkGrey</material>

File: omni_base_description/urdf/sensors/sick_tim551_laser.urdf.xacro (robot description, xacro)
@@ -28,5 +28,5 @@
         <origin xyz="0 0 0" rpy="0 0 0" />
         <geometry>
-          <mesh filename="package://omni_base_description/meshes/sensors/sick_tim551.stl" scale="1 1 1"/>
+          <mesh filename="file://$(find omni_base_description)/meshes/sensors/sick_tim551.stl" scale="1 1 1"/>
         </geometry>
         <material name="DarkGrey"/>

File: omni_base_description/urdf/sensors/sick_tim561_laser.gazebo.xacro (robot description, xacro)
@@ -16,9 +16,11 @@
   <xacro:macro name="sick_tim561_laser_gazebo" params="name ros_topic update_rate min_angle max_angle">
     <gazebo reference="${name}_link">
-      <sensor type="gpu_ray" name="${name}">
+      <sensor type="gpu_lidar" name="${name}">
         <pose>0 0 0 0 0 0</pose>
         <update_rate>${update_rate}</update_rate>
         <visualize>true</visualize>
-        <ray>
+        <topic>${ros_topic}</topic>
+        <gz_frame_id>${name}_link</gz_frame_id>
+        <lidar>
           <scan>
             <horizontal>
@@ -41,11 +43,4 @@
           </noise>
         </ray>
-      	<plugin name="${name}" filename="libgazebo_ros_ray_sensor.so">
-          <ros>
-      	    <remapping>~/out:=${ros_topic}</remapping>
-          </ros>
-          <output_type>sensor_msgs/LaserScan</output_type>
-      	  <frame_name>${name}_link</frame_name>
-        </plugin>
       </sensor>
       <material>Gazebo/DarkGrey</material>

File: omni_base_description/urdf/sensors/sick_tim561_laser.urdf.xacro (robot description, xacro)
@@ -28,5 +28,5 @@
         <origin xyz="0 0 0" rpy="0 0 0" />
         <geometry>
-          <mesh filename="package://omni_base_description/meshes/sensors/sick_tim551.stl" scale="1 1 1"/>
+          <mesh filename="file://$(find omni_base_description)/meshes/sensors/sick_tim551.stl" scale="1 1 1"/>
         </geometry>
         <material name="DarkGrey"/>

File: omni_base_description/urdf/sensors/sick_tim571_laser.gazebo.xacro (robot description, xacro)
@@ -16,9 +16,11 @@
   <xacro:macro name="sick_tim571_laser_gazebo" params="name ros_topic update_rate min_angle max_angle">
     <gazebo reference="${name}_link">
-      <sensor type="gpu_ray" name="${name}">
+      <sensor type="gpu_lidar" name="${name}">
         <pose>0 0 0 0 0 0</pose>
         <update_rate>${update_rate}</update_rate>
         <visualize>true</visualize>
-        <ray>
+        <topic>${ros_topic}</topic>
+        <gz_frame_id>${name}_link</gz_frame_id>
+        <lidar>
           <scan>
             <horizontal>
@@ -40,12 +42,5 @@
             <stddev>0.01</stddev>
           </noise>
-        </ray>
-      	<plugin name="${name}" filename="libgazebo_ros_ray_sensor.so">
-          <ros>
-      	    <remapping>~/out:=${ros_topic}</remapping>
-          </ros>
-          <output_type>sensor_msgs/LaserScan</output_type>
-      	  <frame_name>${name}_link</frame_name>
-        </plugin>
+        </lidar>
       </sensor>
       <material>Gazebo/DarkGrey</material>

File: omni_base_description/urdf/sensors/sick_tim571_laser.urdf.xacro (robot description, xacro)
@@ -28,5 +28,5 @@
         <origin xyz="0 0 0" rpy="0 0 0" />
         <geometry>
-          <mesh filename="package://omni_base_description/meshes/sensors/sick_tim551.stl" scale="1 1 1"/>
+          <mesh filename="file://$(find omni_base_description)/meshes/sensors/sick_tim551.stl" scale="1 1 1"/>
         </geometry>
         <material name="DarkGrey"/>

File: omni_base_description/urdf/wheels/wheel.urdf.xacro (robot description, xacro)
@@ -30,8 +30,8 @@
         <geometry>
           <xacro:if value="${frontal_reflect == 1}">
-            <mesh filename="package://omni_base_description/meshes/wheels/suspension_front_link.stl" scale="1 ${sagital_reflect} 1"/>
+            <mesh filename="file://$(find omni_base_description)/meshes/wheels/suspension_front_link.stl" scale="1 ${sagital_reflect} 1"/>
           </xacro:if>
           <xacro:unless value="${frontal_reflect == 1}">
-            <mesh filename="package://omni_base_description/meshes/wheels/suspension_rear_link.stl" scale="1 ${sagital_reflect} 1"/>
+            <mesh filename="file://$(find omni_base_description)/meshes/wheels/suspension_rear_link.stl" scale="1 ${sagital_reflect} 1"/>
           </xacro:unless>
         </geometry>
@@ -44,8 +44,8 @@
         <geometry>
           <xacro:if value="${frontal_reflect == 1}">
-            <mesh filename="package://omni_base_description/meshes/wheels/suspension_front_link.stl" scale="1 ${sagital_reflect} 1"/>
+            <mesh filename="file://$(find omni_base_description)/meshes/wheels/suspension_front_link.stl" scale="1 ${sagital_reflect} 1"/>
           </xacro:if>
           <xacro:unless value="${frontal_reflect == 1}">
-            <mesh filename="package://omni_base_description/meshes/wheels/suspension_rear_link.stl" scale="1 ${sagital_reflect} 1"/>
+            <mesh filename="file://$(find omni_base_description)/meshes/wheels/suspension_rear_link.stl" scale="1 ${sagital_reflect} 1"/>
           </xacro:unless>
         </geometry>
@@ -71,5 +71,5 @@
         <origin xyz="0 0 0" rpy="0 0 0" />
         <geometry>
-          <mesh filename="package://omni_base_description/meshes/wheels/wheel_link.stl" scale="1 1 ${sagital_reflect}"/>
+          <mesh filename="file://$(find omni_base_description)/meshes/wheels/wheel_link.stl" scale="1 1 ${sagital_reflect}"/>
         </geometry>
         <material name="DarkGrey"/>
